File: GPS.kicad_pcb (KiCad board)
At the start: 4 copper layers, 43 x 34 mm, 29 parts, among them J1 SMA, J2 Conn_01x07, U1 TXS0108EPW, U101 AP2112K-3.3, U3 LC29H

Commit message: Clean up area underneath antenna
Parts:
- renumbered C13 to C1, C5 to C10, C9 to C11, C3 to C12, C1 to C13, C2 to C14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
Routing:
- net GND: vias 129 -> 133
